File: my_pcb/my pcb.kicad_sch (KiCad schematic)
At the start: 5 parts, among them U1 ATmega32U4-A

Commit message: Finished Schem
Parts:
- added C1, C2, C7: 10uF, Capacitor_SMD:C_0805_2012Metric, symbol Device:C_Small
- added C4, C5, C6: 0.1uF, Capacitor_SMD:C_0805_2012Metric, symbol Device:C_Small
- added D1, D2, D3, D4: D_Small, Diode_SMD:D_SOD-123, symbol Device:D_Small
- added F1: 500mA, Fuse:Fuse_1206_3216Metric, symbol Device:Polyfuse
- added MX1, MX2, MX3, MX4: MX-NoLED, Button_Switch_Keyboard:SW_Cherry_MX_1.00u_PCB, symbol MX_Alps_Hybrid:MX-NoLED
- added R1: 10k, Resistor_SMD:R_0805_2012Metric, symbol Device:R_Small
- added SW1: SW_Push, random-keyboard-parts:SKQG-1155865, symbol Switch:SW_Push
- added USB1: Molex-0548190589, random-keyboard-parts:Molex-0548190589, symbol random-keyboard-parts:Molex-0548190589
- added Y1: 16Mhz, Crystal:Crystal_SMD_3225-4Pin_3.2x2.5mm, symbol Device:Crystal_GND24_Small
- C3: renamed from C1; value C_Small -> 1uF; footprint (none) -> Capacitor_SMD:C_0805_2012Metric
- R2, R3, R4: renamed from R?; footprint (none) -> Resistor_SMD:R_0805_2012Metric
Connections:
- net +5V: now also U1.7 (VBUS), C4.1, C5.1, C6.1, C7.1, F1.2, R1.1
- net GND: now also C3.2, C1.1, C2.1, C4.2, C5.2, C6.2, C7.2, SW1.1, USB1.1 (GND), Y1.2, Y1.4
- net D-: now reaches R3.2
- net D-: now also USB1.4 (D-)
- net D+: now reaches R2.2
- net D+: now also USB1.3 (D+)
- net at U1.13 (~{RESET}): now also R1.2, SW1.2
- net at U1.16 (XTAL2): now also C2.2, Y1.3
- net at U1.17 (XTAL1): now also C1.2, Y1.1
- new net: D2.2 (A), MX2.2 (ROW)
- new net: D1.2 (A), MX1.2 (ROW)
- new net: F1.1, USB1.5 (VBUS)
- new net: D3.2 (A), MX3.2 (ROW)
- new net: D4.2 (A), MX4.2 (ROW)
- new net COL0: MX1.1 (COL), MX3.1 (COL)
- new net COL1: MX2.1 (COL), MX4.1 (COL)
- new net ROW0: D1.1 (K), D2.1 (K)
- new net ROW1: D3.1 (K), D4.1 (K)
